File: final-forme.sch (KiCad schematic (older format))
At the start: 14 parts

Commit message: pcb
partial routing
Parts:
- added D1, D10, D100, D11, D12, D13, D14, D15, D16, D17, D18, D19, D2, D20, D21, D22, D23, D24, D25, D26, D27, D28, D29, D3, D30, D31, D32, D33, D34, D35, D36, D37, D38, D39, D4, D40, D41, D42, D43, D44, D45, D46, D47, D48, D49, D5, D50, D51, D52, D53, D54, D55, D56, D57, D58, D59, D6, D60, D61, D62, D63, D64, D65, D66, D67, D68, D69, D7, D70, D71, D72, D73, D74, D75, D76, D77, D78, D79, D8, D80, D81, D82, D83, D84, D85, D86, D87, D88, D89, D9, D90, D91, D92, D93, D94, D95, D96, D97, D98, D99: D_Small, Diode_SMD:D_SOD-123, symbol Device:D_Small
- added F1: 500mA, Fuse:Fuse_1206_3216Metric_Pad1.42x1.75mm_HandSolder, symbol Device:Polyfuse_Small
- added MX1, MX10, MX11, MX12, MX13, MX14, MX15, MX16, MX17, MX18, MX19, MX2, MX20, MX21, MX22, MX23, MX24, MX25, MX26, MX27, MX28, MX29, MX3, MX31, MX32, MX33, MX34, MX36, MX37, MX38, MX39, MX4, MX40, MX41, MX42, MX43, MX44, MX45, MX46, MX47, MX49, MX5, MX50, MX51, MX52, MX54, MX55, MX56, MX57, MX58, MX59, MX6, MX60, MX61, MX62, MX63, MX64, MX66, MX67, MX68, MX69, MX7, MX72, MX73, MX74, MX75, MX76, MX77, MX78, MX79, MX8, MX80, MX81, MX83, MX84, MX85, MX86, MX87, MX9, MX92, MX93, MX94, MX95, MX96, MX97, MX99: MX-NoLED, MX_Alps_Hybrid:MX-1U-NoLED, symbol MX_Alps_Hybrid:MX-NoLED
- added MX100, MX70: MX-NoLED, MX_Alps_Hybrid:MX-2U-NoLED-Vertical, symbol MX_Alps_Hybrid:MX-NoLED
- added MX30, MX98: MX-NoLED, MX_Alps_Hybrid:MX-2U-NoLED, symbol MX_Alps_Hybrid:MX-NoLED
- added MX35, MX48: MX-NoLED, MX_Alps_Hybrid:MX-1.5U-NoLED, symbol MX_Alps_Hybrid:MX-NoLED
- added MX53, MX82: MX-NoLED, MX_Alps_Hybrid:MX-1.75U-NoLED, symbol MX_Alps_Hybrid:MX-NoLED
- added MX65, MX71: MX-NoLED, MX_Alps_Hybrid:MX-2.25U-NoLED, symbol MX_Alps_Hybrid:MX-NoLED
- added MX88, MX89, MX90: MX-NoLED, MX_Alps_Hybrid:MX-1.25U-NoLED, symbol MX_Alps_Hybrid:MX-NoLED
- added MX91: MX-NoLED, MX_Alps_Hybrid:MX-6.25U-NoLED, symbol MX_Alps_Hybrid:MX-NoLED
- added R5, R6: 5.1k, Resistor_SMD:R_1206_3216Metric_Pad1.30x1.75mm_HandSolder, symbol Device:R_Small_US
- added USB1: USB4085-GF-A, USB-C:USB4085-GF-A, symbol USB-C:USB4085-GF-A
- C1, C2, C3, C4, C5, C6, C7: renamed from C?; footprint (none) -> Capacitor_SMD:C_1206_3216Metric_Pad1.33x1.80mm_HandSolder
- R1, R2, R3, R4: renamed from R?; footprint (none) -> Resistor_SMD:R_1206_3216Metric_Pad1.30x1.75mm_HandSolder
- SW1: renamed from SW?; footprint (none) -> random-keyboard-parts:SKQG-1155865
- Y1: renamed from Y?; footprint (none) -> Crystal:Crystal_SMD_3225-4Pin_3.2x2.5mm_HandSoldering
- gave numbers to parts that had none: 1
Connections:
- net +5V: now also F1.1
- net D+: now also USB1.A6 (D+1), USB1.B6 (D+2)
- net D-: now also USB1.A7 (D-1), USB1.B7 (D-2)
- net GND: now also R5.1, R6.1, USB1.A1 (GND), USB1.A12 (GND), USB1.B1 (GND), USB1.B12 (GND), USB1.SHIELD
- new net: F1.2, USB1.A4 (Vbus), USB1.A9 (Vbus), USB1.B4 (Vbus), USB1.B9 (Vbus)
- new net: R6.2, USB1.A5 (CC1)
- new net: R5.2, USB1.B5 (CC2)
- new net: D1.2 (A), MX1.2 (ROW)
- new net: D2.2 (A), MX2.2 (ROW)
- new net: D3.2 (A), MX3.2 (ROW)
- new net: D4.2 (A), MX4.2 (ROW)
- new net: D5.2 (A), MX5.2 (ROW)
- new net: D6.2 (A), MX6.2 (ROW)
- new net: D7.2 (A), MX7.2 (ROW)
- new net: D8.2 (A), MX8.2 (ROW)
- new net: D9.2 (A), MX9.2 (ROW)
- new net: D10.2 (A), MX10.2 (ROW)
- new net: D11.2 (A), MX11.2 (ROW)
- new net: D12.2 (A), MX12.2 (ROW)
- new net: D13.2 (A), MX13.2 (ROW)
- new net: D14.2 (A), MX14.2 (ROW)
- new net: D15.2 (A), MX15.2 (ROW)
- new net: D17.2 (A), MX17.2 (ROW)
- new net: D18.2 (A), MX18.2 (ROW)
- new net: D19.2 (A), MX19.2 (ROW)
- new net: D20.2 (A), MX20.2 (ROW)
- new net: D21.2 (A), MX21.2 (ROW)
- new net: D22.2 (A), MX22.2 (ROW)
- new net: D23.2 (A), MX23.2 (ROW)
- new net: D24.2 (A), MX24.2 (ROW)
- new net: D25.2 (A), MX25.2 (ROW)
- new net: D26.2 (A), MX26.2 (ROW)
- new net: D27.2 (A), MX27.2 (ROW)
- new net: D28.2 (A), MX28.2 (ROW)
- new net: D29.2 (A), MX29.2 (ROW)
- new net: D30.2 (A), MX30.2 (ROW)
- new net: D31.2 (A), MX31.2 (ROW)
- new net: D32.2 (A), MX32.2 (ROW)
- new net: D33.2 (A), MX33.2 (ROW)
- new net: D16.2 (A), MX16.2 (ROW)
- new net: D35.2 (A), MX35.2 (ROW)
- new net: D36.2 (A), MX36.2 (ROW)
- new net: D37.2 (A), MX37.2 (ROW)
- new net: D38.2 (A), MX38.2 (ROW)
- new net: D39.2 (A), MX39.2 (ROW)
- new net: D40.2 (A), MX40.2 (ROW)
- new net: D41.2 (A), MX41.2 (ROW)
- new net: D42.2 (A), MX42.2 (ROW)
- new net: D43.2 (A), MX43.2 (ROW)
- new net: D44.2 (A), MX44.2 (ROW)
- new net: D45.2 (A), MX45.2 (ROW)
- new net: D46.2 (A), MX46.2 (ROW)
- new net: D47.2 (A), MX47.2 (ROW)
- new net: D48.2 (A), MX48.2 (ROW)
- new net: D49.2 (A), MX49.2 (ROW)
- new net: D50.2 (A), MX50.2 (ROW)
- new net: D51.2 (A), MX51.2 (ROW)
- new net: D53.2 (A), MX53.2 (ROW)
- new net: D54.2 (A), MX54.2 (ROW)
- new net: D55.2 (A), MX55.2 (ROW)
- new net: D56.2 (A), MX56.2 (ROW)
- new net: D57.2 (A), MX57.2 (ROW)
- new net: D58.2 (A), MX58.2 (ROW)
- new net: D59.2 (A), MX59.2 (ROW)
- new net: D60.2 (A), MX60.2 (ROW)
- new net: D61.2 (A), MX61.2 (ROW)
- new net: D62.2 (A), MX62.2 (ROW)
- new net: D63.2 (A), MX63.2 (ROW)
- new net: D64.2 (A), MX64.2 (ROW)
- new net: D65.2 (A), MX65.2 (ROW)
- new net: D66.2 (A), MX66.2 (ROW)
- new net: D67.2 (A), MX67.2 (ROW)
- new net: D68.2 (A), MX68.2 (ROW)
- new net: D69.2 (A), MX69.2 (ROW)
- new net: D71.2 (A), MX71.2 (ROW)
- new net: D72.2 (A), MX72.2 (ROW)
- new net: D73.2 (A), MX73.2 (ROW)
- new net: D74.2 (A), MX74.2 (ROW)
- new net: D75.2 (A), MX75.2 (ROW)
- new net: D76.2 (A), MX76.2 (ROW)
- new net: D77.2 (A), MX77.2 (ROW)
- new net: D78.2 (A), MX78.2 (ROW)
- new net: D79.2 (A), MX79.2 (ROW)
- new net: D80.2 (A), MX80.2 (ROW)
- new net: D81.2 (A), MX81.2 (ROW)
- new net: D82.2 (A), MX82.2 (ROW)
- new net: D83.2 (A), MX83.2 (ROW)
- new net: D84.2 (A), MX84.2 (ROW)
- new net: D85.2 (A), MX85.2 (ROW)
- new net: D86.2 (A), MX86.2 (ROW)
- new net: D87.2 (A), MX87.2 (ROW)
- new net: D34.2 (A), MX34.2 (ROW)
- new net: D52.2 (A), MX52.2 (ROW)
- new net: D70.2 (A), MX70.2 (ROW)
- new net: D88.2 (A), MX88.2 (ROW)
- new net: D89.2 (A), MX89.2 (ROW)
- new net: D90.2 (A), MX90.2 (ROW)
- new net: D91.2 (A), MX91.2 (ROW)
- new net: D92.2 (A), MX92.2 (ROW)
- new net: D93.2 (A), MX93.2 (ROW)
- new net: D94.2 (A), MX94.2 (ROW)
- new net: D95.2 (A), MX95.2 (ROW)
- new net: D96.2 (A), MX96.2 (ROW)
- new net: D97.2 (A), MX97.2 (ROW)
- new net: D98.2 (A), MX98.2 (ROW)
- new net: D99.2 (A), MX99.2 (ROW)
- new net: D100.2 (A), MX100.2 (ROW)
- new net COL0: MX1.1 (COL), MX17.1 (COL), MX35.1 (COL), MX53.1 (COL), MX71.1 (COL), MX88.1 (COL)
- new net COL1: MX18.1 (COL), MX2.1 (COL), MX36.1 (COL), MX54.1 (COL), MX72.1 (COL), MX89.1 (COL)
- new net COL10: MX11.1 (COL), MX27.1 (COL), MX45.1 (COL), MX63.1 (COL), MX81.1 (COL), MX94.1 (COL)
- new net COL11: MX12.1 (COL), MX28.1 (COL), MX46.1 (COL), MX64.1 (COL), MX82.1 (COL), MX95.1 (COL)
- new net COL12: MX13.1 (COL), MX29.1 (COL), MX47.1 (COL), MX65.1 (COL), MX83.1 (COL), MX96.1 (COL)
- new net COL13: MX14.1 (COL), MX30.1 (COL), MX48.1 (COL), MX66.1 (COL), MX84.1 (COL), MX97.1 (COL)
- new net COL14: MX15.1 (COL), MX31.1 (COL), MX49.1 (COL), MX67.1 (COL), MX85.1 (COL), MX98.1 (COL)
- new net COL15: MX16.1 (COL), MX32.1 (COL), MX50.1 (COL), MX68.1 (COL), MX86.1 (COL), MX99.1 (COL)
- new net COL16: MX100.1 (COL), MX33.1 (COL), MX51.1 (COL), MX69.1 (COL), MX87.1 (COL)
- new net COL17: MX34.1 (COL), MX52.1 (COL), MX70.1 (COL)
- new net COL2: MX19.1 (COL), MX3.1 (COL), MX37.1 (COL), MX55.1 (COL), MX73.1 (COL), MX90.1 (COL)
- new net COL3: MX20.1 (COL), MX38.1 (COL), MX4.1 (COL), MX56.1 (COL), MX74.1 (COL)
- new net COL4: MX21.1 (COL), MX39.1 (COL), MX5.1 (COL), MX57.1 (COL), MX75.1 (COL)
- new net COL5: MX22.1 (COL), MX40.1 (COL), MX58.1 (COL), MX6.1 (COL), MX76.1 (COL), MX91.1 (COL)
- new net COL6: MX23.1 (COL), MX41.1 (COL), MX59.1 (COL), MX7.1 (COL), MX77.1 (COL)
- new net COL7: MX24.1 (COL), MX42.1 (COL), MX60.1 (COL), MX78.1 (COL), MX8.1 (COL)
- new net COL8: MX25.1 (COL), MX43.1 (COL), MX61.1 (COL), MX79.1 (COL), MX9.1 (COL), MX92.1 (COL)
- new net COL9: MX10.1 (COL), MX26.1 (COL), MX44.1 (COL), MX62.1 (COL), MX80.1 (COL), MX93.1 (COL)
- new net ROW0: D1.1 (K), D10.1 (K), D11.1 (K), D12.1 (K), D13.1 (K), D14.1 (K), D15.1 (K), D16.1 (K), D2.1 (K), D3.1 (K), D4.1 (K), D5.1 (K), D6.1 (K), D7.1 (K), D8.1 (K), D9.1 (K)
- new net ROW1: D17.1 (K), D18.1 (K), D19.1 (K), D20.1 (K), D21.1 (K), D22.1 (K), D23.1 (K), D24.1 (K), D25.1 (K), D26.1 (K), D27.1 (K), D28.1 (K), D29.1 (K), D30.1 (K), D31.1 (K), D32.1 (K), D33.1 (K), D34.1 (K)
- new net ROW2: D35.1 (K), D36.1 (K), D37.1 (K), D38.1 (K), D39.1 (K), D40.1 (K), D41.1 (K), D42.1 (K), D43.1 (K), D44.1 (K), D45.1 (K), D46.1 (K), D47.1 (K), D48.1 (K), D49.1 (K), D50.1 (K), D51.1 (K), D52.1 (K)
- new net ROW3: D53.1 (K), D54.1 (K), D55.1 (K), D56.1 (K), D57.1 (K), D58.1 (K), D59.1 (K), D60.1 (K), D61.1 (K), D62.1 (K), D63.1 (K), D64.1 (K), D65.1 (K), D66.1 (K), D67.1 (K), D68.1 (K), D69.1 (K), D70.1 (K)
- new net ROW4: D71.1 (K), D72.1 (K), D73.1 (K), D74.1 (K), D75.1 (K), D76.1 (K), D77.1 (K), D78.1 (K), D79.1 (K), D80.1 (K), D81.1 (K), D82.1 (K), D83.1 (K), D84.1 (K), D85.1 (K), D86.1 (K), D87.1 (K)
- new net ROW5: D100.1 (K), D88.1 (K), D89.1 (K), D90.1 (K), D91.1 (K), D92.1 (K), D93.1 (K), D94.1 (K), D95.1 (K), D96.1 (K), D97.1 (K), D98.1 (K), D99.1 (K)
Other:
- moved on the sheet: C1, C2, C3, C4, C5, C6, C7, R1, R2, R3, R4, SW1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
